File: BaofengInterface/BaofengInterface.sch (KiCad schematic (older format))
At the start: 9 parts

Commit message: PCB layou finish
Parts:
- removed JP? (x2): Jumper_NO_Small, symbol Jumper_NO_Small
- added J5: CONN_01X03, Pin_Headers:Pin_Header_Straight_1x03_Pitch2.54mm, symbol CONN_01X03
- C1: renamed from C?; footprint (none) -> Capacitors_THT:C_Disc_D4.7mm_W2.5mm_P5.00mm; MFN (none) -> TDK Corporation; MFRPN (none) -> FG28X5R1H105KRT06; Supplier1_Link (none) -> https://www.digikey.com/product-detail/en/tdk-corporation/F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; Supplier1_PN (none) -> 445-173579-1-ND
- J1: renamed from J?; footprint (none) -> Pin_Headers:Pin_Header_Straight_1x06_Pitch2.54mm
- J2: renamed from J?; footprint (none) -> Pin_Headers:Pin_Header_Straight_1x04_Pitch2.54mm
- J3, J4: renamed from J?; footprint (none) -> SJ1-352XN:SJ1-352XN
- Q1: renamed from Q?; footprint (none) -> TO_SOT_Packages_THT:TO-92_Inline_Narrow_Oval
- R1: renamed from R?; footprint (none) -> Resistors_THT:R_Axial_DIN0207_L6.3mm_D2.5mm_P2.54mm_Vertical; CF14JT1K00 (none) -> MFRPN; MFN (none) -> Stackpole Electronics Inc.; Supplier1_Link (none) -> https://www.digikey.com/product-detail/en/stackpole-electro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; Supplier1_PN (none) -> CF14JT1K00CT-ND
Connections:
- net SERIAL_RX: now also J2.2 (P2); no longer J2.3 (P3)
- net SERIAL_TX: now also J2.3 (P3); no longer J2.2 (P2)
- net TX_AUDIO: now also J5.2 (P2)
- net TX_LEFT+: now also J5.3 (P3)
- net TX_RIGHT+: now also J5.1 (P1)
Other:
- moved on the sheet: C1, J1, J2, J3, J4, Q1, R1
